File: amg8833.brd (EAGLE design)
At the start: 25.6 x 34.2 mm, 19 parts, among them Q1 BSN20,215, U1 AMG8833

Commit message: fixes #1, #2
Parts:
- added R6: 10k, rcl:R0603
- J3: device SparkFun-Connectors:1X03_LONGPADS -> SparkFun-Connectors:SCREWTERMINAL-3.5MM-3-NS
- R1, R2: value 4k7 -> 10k
- moved J3 1.01 mm to (-3.50, 10.0)
- moved R2 0.25 mm to (7.50, 1.25)
Connections:
- net +3V3: now also R6.2
- net AMGINT: now also R6.1
- net NEOPIX3V3: now also J1.5; no longer J1.6
Routing:
- net +3V3: track 41.5 -> 44.0 mm
- net NEOPIX3V3: track 4.68 -> 6.58 mm
- net AMGINT: track 8.83 -> 10.1 mm, vias 0 -> 1
- net MEOPIXOUT: track 21.5 -> 22.2 mm
- net SCL: track 12.2 -> 11.6 mm
- net SDA: track 10.5 -> 11.1 mm

Commit message: silkscreen/naming fixes
Parts:
- R3: value 4k7 -> 10k
- R4: value 20 -> 4k7
- R5: value 4k7 -> 20
- R6: value 10k -> 4k7
- moved R3 17.2 mm to (7.50, -1.00), turned to 0 degrees
- moved R6 17.2 mm to (-9.00, 4.00), turned to 270 degrees
- moved R4 2.00 mm to (-2.00, 6.00)
- moved R5 2.00 mm to (-2.00, 4.00)
- renumbered C5 to C3, C6 to C2, C7 to C1
Connections:
- net +5V: now also R4.2; no longer R5.2
- net AMGINT: now also R3.1; no longer R6.1
- net GND: now also R5.2; no longer R4.2
- net N$6: now also R5.1; no longer R4.1
- net NEOPIX3V3: now also R6.1; no longer R3.1
- net NEOPIX5V: now also R4.1; no longer R5.1
