File: amg8833.brd (EAGLE design)
At the start: 25.6 x 34.2 mm, 20 parts, among them Q1 BSN20,215, U1 AMG8833

Commit message: 3d stuff
Parts:
- D1, D2, D3: device SparkFun-LED:WS2812B -> jonas_SparkFun-LED:WS2812B
- J1, J2: device SparkFun-Connectors:1X08_LOCK_NO_SILK -> jonas_Sparkfun-Connectors:1X08_LOCK_NO_SILK
- J3: device SparkFun-Connectors:SCREWTERMINAL-3.5MM-3-NS -> jonas_Sparkfun-Connectors:SCREWTERMINAL-3.5MM-3-NS
- JP1: value (none) -> JUMPER-SMT_2_NC_TRACE; device SparkFun-Jumpers:SMT-JUMPER_2_NC_TRACE_SILK -> jonas_SparkFun_Jumper:SMT-JUMPER_2_NC_TRACE_SILK
- JP2: device SparkFun-Jumpers:SMT-JUMPER_3_1-NC_TRACE_SILK -> jonas_SparkFun_Jumper:SMT-JUMPER_3_1-NC_TRACE_SILK
- LOGO1: value OSHW-LOGOM -> OSHW-LOGO; device SparkFun-Aesthetics:OSHW-LOGO-M -> jonas_SparkFun-Aesthetics:OSHW-LOGO-M
Changed lines of the file:
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@@
 <?xml version="1.0" encoding="utf-8"?>
 <!DOCTYPE eagle SYSTEM "eagle.dtd">
-<eagle version="9.0.1">
+<eagle version="9.1.0">
 <drawing>
 <settings>
@@
 </layers>
 <board>
-<fusionsync huburn="a.cGVyc29uYWw6dWUyOTRlNWI0" projecturn="a.cGVyc29uYWw6dWUyOTRlNWI0IzIwMTgwNjIyMTM3MzUxMTgx" f3durn="urn:adsk.wipprod:dm.lineage:VgF9cCN1SuO1Fo5ZokwAeA" pcbguid="a747b205-4403-415a-b58b-43fccb9cd7a5" lastpulledtime="" lastsyncedchangeguid="99fbabed-0915-d1c1-0f20-aca28310aa02"/>
+<fusionsync huburn="a.cGVyc29uYWw6dWUyOTRlNWI0" projecturn="a.cGVyc29uYWw6dWUyOTRlNWI0IzIwMTgwNjIyMTM3MzUxMTgx" f3durn="urn:adsk.wipprod:dm.lineage:VgF9cCN1SuO1Fo5ZokwAeA" pcbguid="a747b205-4403-415a-b58b-43fccb9cd7a5" lastpulledtime="" lastsyncedchangeguid="670e9adf-07a5-ee30-4a8e-eb4bc8a32c00"/>
 <plain>
 <wire x1="-12.8" y1="-17.54" x2="12.8" y2="-17.54" width="0" layer="20"/>
@@
 <param name="checkStop" value="0"/>
 <param name="checkValues" value="0"/>
+<param name="checkNames" value="1"/>
+<param name="checkWireStubs" value="1"/>
+<param name="checkPolygonWidth" value="0"/>
 <param name="useDiameter" value="13"/>
 <param name="maxErrors" value="50"/>
@@
 <attribute name="VALUE" x="-2.365" y="0.095" size="1.27" layer="28" rot="MR0"/>
 </element>
-<element name="D1" library="SparkFun-LED" library_urn="urn:adsk.eagle:library:529" package="WS2812B" package3d_urn="urn:adsk.eagle:package:39369/1" value="WS2812B" x="-6" y="-13" smashed="yes" rot="R270">
-<attribute name="PROD_ID" value="DIO-12503" x="-6" y="-13" size="1.778" layer="27" rot="R270" display="off"/>
-</element>
-<element name="D2" library="SparkFun-LED" library_urn="urn:adsk.eagle:library:529" package="WS2812B" package3d_urn="urn:adsk.eagle:package:39369/1" value="WS2812B" x="0" y="-13" smashed="yes" rot="R270">
-<attribute name="PROD_ID" value="DIO-12503" x="0" y="-13" size="1.778" layer="27" rot="R270" display="off"/>
-</element>
-<element name="D3" library="SparkFun-LED" library_urn="urn:adsk.eagle:library:529" package="WS2812B" package3d_urn="urn:adsk.eagle:package:39369/1" value="WS2812B" x="6" y="-13" smashed="yes" rot="R270">
-<attribute name="PROD_ID" value="DIO-12503" x="6" y="-13" size="1.778" layer="27" rot="R270" display="off"/>
-</element>
+<element name="D1" library="jonas_SparkFun-LED" library_urn="urn:adsk.eagle:library:3855694" package="WS2812B" package3d_urn="urn:adsk.eagle:package:3855696/2" value="WS2812B" x="-6" y="-13" smashed="yes" rot="R270"/>
+<element name="D2" library="jonas_SparkFun-LED" library_urn="urn:adsk.eagle:library:3855694" package="WS2812B" package3d_urn="urn:adsk.eagle:package:3855696/2" value="WS2812B" x="0" y="-13" smashed="yes" rot="R270"/>
+<element name="D3" library="jonas_SparkFun-LED" library_urn="urn:adsk.eagle:library:3855694" package="WS2812B" package3d_urn="urn:adsk.eagle:package:3855696/2" value="WS2812B" x="6" y="-13" smashed="yes" rot="R270"/>
 <element name="Q1" library="jonas_mosfet" library_urn="urn:adsk.eagle:library:2195717" package="BSN20_215" package3d_urn="urn:adsk.eagle:package:2195720/4" value="BSN20,215" x="-6" y="4" smashed="yes" rot="MR90">
 <attribute name="AVAILABILITY" value="Good" x="-6" y="4" size="1.778" layer="28" rot="MR90" display="off"/>
@@
 <attribute name="VALUE" x="-2.635" y="7.905" size="1.27" layer="28" rot="MR180"/>
 </element>
-<element name="J1" library="SparkFun-Connectors" library_urn="urn:adsk.eagle:library:513" package="1X08_LOCK_NO_SILK" package3d_urn="urn:adsk.eagle:package:38147/1" value="" x="-11.43" y="-8.89" smashed="yes" rot="R90">
+<element name="J1" library="jonas_Sparkfun-Connectors" library_urn="urn:adsk.eagle:library:3855661" package="1X08_LOCK_NO_SILK" package3d_urn="urn:adsk.eagle:package:3855663/2" value="" x="-11.43" y="-8.89" smashed="yes" rot="R90">
 <attribute name="VALUE" x="-9.398" y="-10.16" size="0.6096" layer="27" font="vector" ratio="20" rot="R90"/>
 </element>
-<element name="J2" library="SparkFun-Connectors" library_urn="urn:adsk.eagle:library:513" package="1X08_LOCK_NO_SILK" package3d_urn="urn:adsk.eagle:package:38147/1" value="" x="11.43" y="-8.89" smashed="yes" rot="R90">
+<element name="J2" library="jonas_Sparkfun-Connectors" library_urn="urn:adsk.eagle:library:3855661" package="1X08_LOCK_NO_SILK" package3d_urn="urn:adsk.eagle:package:3855663/2" value="" x="11.43" y="-8.89" smashed="yes" rot="R90">
 <attribute name="VALUE" x="13.462" y="-10.16" size="0.6096" layer="27" font="vector" ratio="20" rot="R90"/>
 </element>
-<element name="JP1" library="SparkFun-Jumpers" library_urn="urn:adsk.eagle:library:528" package="SMT-JUMPER_2_NC_TRACE_SILK" package3d_urn="urn:adsk.eagle:package:39281/1" value="" x="-7" y="-6" smashed="yes" rot="MR90">
+<element name="JP1" library="jonas_SparkFun_Jumper" library_urn="urn:adsk.eagle:library:3855711" package="SMT-JUMPER_2_NC_TRACE_SILK" package3d_urn="urn:adsk.eagle:package:3855718/2" value="JUMPER-SMT_2_NC_TRACE" x="-7" y="-6" smashed="yes" rot="MR90">
 <attribute name="NAME" x="-7" y="-4.607" size="0.8128" layer="26" font="vector" ratio="15" rot="MR0" align="bottom-center"/>
 <attribute name="VALUE" x="-8.143" y="-6" size="0.6096" layer="28" font="vector" ratio="20" rot="MR90" align="top-center"/>
 </element>
-<element name="JP2" library="SparkFun-Jumpers" library_urn="urn:adsk.eagle:library:528" package="SMT-JUMPER_3_1-NC_TRACE_SILK" package3d_urn="urn:adsk.eagle:package:39288/1" value="" x="-4" y="-8" smashed="yes" rot="MR180">
+<element name="JP2" library="jonas_SparkFun_Jumper" library_urn="urn:adsk.eagle:library:3855711" package="SMT-JUMPER_3_1-NC_TRACE_SILK" package3d_urn="urn:adsk.eagle:package:3855713/2" value="" x="-4" y="-8" smashed="yes" rot="MR180">
 <attribute name="NAME" x="-4" y="-9.143" size="0.8128" layer="26" font="vector" ratio="20" rot="MR180" align="bottom-center"/>
 <attribute name="VALUE" x="-4" y="-6.857" size="0.6096" layer="28" font="vector" ratio="20" rot="MR180" align="top-center"/>
 </element>
-<element name="LOGO1" library="SparkFun-Aesthetics" library_urn="urn:adsk.eagle:library:507" package="OSHW-LOGO-M" package3d_urn="urn:adsk.eagle:package:37126/1" value="OSHW-LOGOM" x="8.8" y="12.66"/>
+<element name="LOGO1" library="jonas_SparkFun-Aesthetics" library_urn="urn:adsk.eagle:library:3855705" package="OSHW-LOGO-M" package3d_urn="urn:adsk.eagle:package:3855707/2" value="OSHW-LOGO" x="8.8" y="12.66"/>
 <element name="R3" library="rcl" library_urn="urn:adsk.eagle:library:334" package="R0603" package3d_urn="urn:adsk.eagle:package:23555/2" value="10k" x="7.5" y="-1" smashed="yes" rot="MR0">
 <attribute name="NAME" x="5.76" y="-0.99" size="0.8128" layer="26" rot="MR0" align="center-left"/>
@@
 <attribute name="VALUE" x="8.135" y="-2.905" size="1.27" layer="28" rot="MR0"/>
 </element>
-<element name="J3" library="SparkFun-Connectors" library_urn="urn:adsk.eagle:library:513" package="SCREWTERMINAL-3.5MM-3-NS" package3d_urn="urn:adsk.eagle:package:38088/1" value="" x="-3.5" y="10" smashed="yes">
-<attribute name="VALUE" x="-1.468" y="5.428" size="0.6096" layer="27" font="vector" ratio="20"/>
-</element>
+<element name="J3" library="jonas_Sparkfun-Connectors" library_urn="urn:adsk.eagle:library:3855661" package="SCREWTERMINAL-3.5MM-3-NS" package3d_urn="urn:adsk.eagle:package:3855668/2" value="" x="-3.5" y="10"/>
 </elements>
 <signals>
@@
 <via x="2" y="4" extent="1-16" drill="0.35"/>
 <via x="0.5" y="5.5" extent="1-16" drill="0.35"/>
+<via x="-6" y="0" extent="1-16" drill="0.35"/>
 <contactref element="J3" pad="1"/>
-<via x="-6" y="0" extent="1-16" drill="0.35"/>
 </signal>
 <signal name="SDA">
@@
 <via x="0.25" y="4" extent="1-16" drill="0.35"/>
 <wire x1="0.25" y1="4" x2="0.25" y2="-4.75" width="0.1524" layer="1"/>
+<wire x1="0.25" y1="4" x2="3.5" y2="7.25" width="0.1524" layer="16"/>
 <contactref element="J3" pad="3"/>
 <wire x1="3.5" y1="7.25" x2="3.5" y2="10" width="0.1524" layer="16"/>
-<wire x1="0.25" y1="4" x2="3.5" y2="7.25" width="0.1524" layer="16"/>
 </signal>
 <signal name="NEOPIXDO">
@@
 </signal>
 </signals>
+<mfgpreviewcolors>
+<mfgpreviewcolor name="soldermaskcolor" color="0xC8008000"/>
+<mfgpreviewcolor name="silkscreencolor" color="0xFFFEFEFE"/>
+<mfgpreviewcolor name="backgroundcolor" color="0x000000"/>
+<mfgpreviewcolor name="coppercolor" color="0xFFFFBF00"/>
+<mfgpreviewcolor name="substratecolor" color="0xFF786E46"/>
+</mfgpreviewcolors>
 <errors>
 </errors>
