File: amg8833.sch (EAGLE design)
At the start: 19 parts, among them Q1 BSN20,215, U1 AMG8833

Commit message: fixes #1, #2
Parts:
- added R6: 10k, rcl:R-EU_R0603
- J3: device SparkFun-Connectors:CONN_03LONGPADS -> SparkFun-Connectors:CONN_03SCREW-NS
- R1, R2: value 4k7 -> 10k
Connections:
- net +3V3: now also R6.2
- net AMGINT: now also R6.1
- net NEOPIX3V3: now also J1.5; no longer J1.6
Changed lines of the file:
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@@
 <parts>
 <part name="+3V2" library="supply1" library_urn="urn:adsk.eagle:library:371" deviceset="+3V3" device=""/>
-<part name="R1" library="rcl" library_urn="urn:adsk.eagle:library:334" deviceset="R-EU_" device="R0603" package3d_urn="urn:adsk.eagle:package:23555/2" value="4k7"/>
-<part name="R2" library="rcl" library_urn="urn:adsk.eagle:library:334" deviceset="R-EU_" device="R0603" package3d_urn="urn:adsk.eagle:package:23555/2" value="4k7"/>
+<part name="R1" library="rcl" library_urn="urn:adsk.eagle:library:334" deviceset="R-EU_" device="R0603" package3d_urn="urn:adsk.eagle:package:23555/2" value="10k"/>
+<part name="R2" library="rcl" library_urn="urn:adsk.eagle:library:334" deviceset="R-EU_" device="R0603" package3d_urn="urn:adsk.eagle:package:23555/2" value="10k"/>
 <part name="U1" library="AMG8833" library_urn="urn:adsk.eagle:library:3739745" deviceset="AMG8833" device="" package3d_urn="urn:adsk.eagle:package:3739748/3"/>
 <part name="+3V1" library="supply1" library_urn="urn:adsk.eagle:library:371" deviceset="+3V3" device=""/>
@@
 <part name="J1" library="SparkFun-Connectors" library_urn="urn:adsk.eagle:library:513" deviceset="CONN_08" device="LOCK_NO_SILK" package3d_urn="urn:adsk.eagle:package:38147/1"/>
 <part name="J2" library="SparkFun-Connectors" library_urn="urn:adsk.eagle:library:513" deviceset="CONN_08" device="LOCK_NO_SILK" package3d_urn="urn:adsk.eagle:package:38147/1"/>
-<part name="J3" library="SparkFun-Connectors" library_urn="urn:adsk.eagle:library:513" deviceset="CONN_03" device="LONGPADS" package3d_urn="urn:adsk.eagle:package:38068/1"/>
 <part name="P+4" library="supply1" library_urn="urn:adsk.eagle:library:371" deviceset="+5V" device=""/>
 <part name="GND5" library="supply1" library_urn="urn:adsk.eagle:library:371" deviceset="GND" device=""/>
@@
 <part name="JP2" library="SparkFun-Jumpers" library_urn="urn:adsk.eagle:library:528" deviceset="JUMPER-SMT_3_1-NC_TRACE" device="_SILK" package3d_urn="urn:adsk.eagle:package:39288/1" value=""/>
 <part name="LOGO1" library="SparkFun-Aesthetics" library_urn="urn:adsk.eagle:library:507" deviceset="OSHW-LOGO" device="M" package3d_urn="urn:adsk.eagle:package:37126/1"/>
+<part name="R6" library="rcl" library_urn="urn:adsk.eagle:library:334" deviceset="R-EU_" device="R0603" package3d_urn="urn:adsk.eagle:package:23555/2" value="10k"/>
+<part name="+3V6" library="supply1" library_urn="urn:adsk.eagle:library:371" deviceset="+3V3" device=""/>
+<part name="J3" library="SparkFun-Connectors" library_urn="urn:adsk.eagle:library:513" deviceset="CONN_03" device="SCREW-NS" package3d_urn="urn:adsk.eagle:package:38088/1"/>
 </parts>
 <sheets>
@@
 <instance part="J1" gate="G$1" x="119.38" y="50.8" rot="MR0"/>
 <instance part="J2" gate="G$1" x="144.78" y="50.8"/>
-<instance part="J3" gate="J$1" x="215.9" y="111.76"/>
 <instance part="P+4" gate="1" x="233.68" y="116.84"/>
 <instance part="GND5" gate="1" x="226.06" y="104.14"/>
@@
 <instance part="JP2" gate="G$1" x="226.06" y="121.92" rot="R90"/>
 <instance part="LOGO1" gate="G$1" x="30.48" y="48.26"/>
+<instance part="R6" gate="G$1" x="81.28" y="45.72" rot="R90"/>
+<instance part="+3V6" gate="G$1" x="81.28" y="55.88"/>
+<instance part="J3" gate="J$1" x="215.9" y="111.76"/>
 </instances>
 <busses>
@@
 <pinref part="+3V5" gate="G$1" pin="+3V3"/>
 </segment>
+<segment>
+<pinref part="R6" gate="G$1" pin="2"/>
+<wire x1="81.28" y1="53.34" x2="81.28" y2="50.8" width="0.1524" layer="91"/>
+<pinref part="+3V6" gate="G$1" pin="+3V3"/>
+</segment>
 </net>
 <net name="GND" class="0">
@@
 </segment>
 <segment>
-<pinref part="J3" gate="J$1" pin="1"/>
 <wire x1="223.52" y1="109.22" x2="226.06" y2="109.22" width="0.1524" layer="91"/>
 <wire x1="226.06" y1="109.22" x2="226.06" y2="106.68" width="0.1524" layer="91"/>
 <pinref part="GND5" gate="1" pin="GND"/>
+<pinref part="J3" gate="J$1" pin="1"/>
 </segment>
 </net>
@@
 <pinref part="J2" gate="G$1" pin="4"/>
 <wire x1="149.86" y1="50.8" x2="152.4" y2="50.8" width="0.1524" layer="91"/>
+</segment>
+<segment>
+<pinref part="R6" gate="G$1" pin="1"/>
+<wire x1="81.28" y1="40.64" x2="81.28" y2="38.1" width="0.1524" layer="91"/>
+<label x="81.28" y="38.1" size="1.016" layer="95" rot="R270" xref="yes"/>
 </segment>
 </net>
@@
 </segment>
 <segment>
-<pinref part="J3" gate="J$1" pin="2"/>
 <wire x1="223.52" y1="111.76" x2="233.68" y2="111.76" width="0.1524" layer="91"/>
 <wire x1="233.68" y1="111.76" x2="233.68" y2="114.3" width="0.1524" layer="91"/>
 <pinref part="P+4" gate="1" pin="+5V"/>
+<pinref part="J3" gate="J$1" pin="2"/>
 </segment>
 </net>
@@
 </segment>
 <segment>
-<label x="111.76" y="55.88" size="1.016" layer="95" rot="R180" xref="yes"/>
-<pinref part="J1" gate="G$1" pin="6"/>
-<wire x1="114.3" y1="55.88" x2="111.76" y2="55.88" width="0.1524" layer="91"/>
+<label x="111.76" y="53.34" size="1.016" layer="95" rot="R180" xref="yes"/>
+<pinref part="J1" gate="G$1" pin="5"/>
+<wire x1="111.76" y1="53.34" x2="114.3" y2="53.34" width="0.1524" layer="91"/>
 </segment>
 </net>
@@
 <net name="MEOPIXOUT" class="0">
 <segment>
-<pinref part="J3" gate="J$1" pin="3"/>
 <wire x1="223.52" y1="114.3" x2="226.06" y2="114.3" width="0.1524" layer="91"/>
 <wire x1="226.06" y1="114.3" x2="226.06" y2="116.84" width="0.1524" layer="91"/>
 <pinref part="JP2" gate="G$1" pin="2"/>
-</segment>
-</net>
+<pinref part="J3" gate="J$1" pin="3"/>
+</segment>
+</net>

Commit message: silkscreen/naming fixes
Parts:
- R3: value 4k7 -> 10k
- R4: value 20 -> 4k7
- R5: value 4k7 -> 20
- R6: value 10k -> 4k7
- renumbered C5 to C3, C6 to C2, C7 to C1
Connections:
- net +5V: now also R4.2; no longer R5.2
- net AMGINT: now also R3.1; no longer R6.1
- net GND: now also R5.2; no longer R4.2
- net N$6: now also R5.1; no longer R4.1
- net NEOPIX3V3: now also R6.1; no longer R3.1
- net NEOPIX5V: now also R4.1; no longer R5.1
Other:
- moved on the sheet: R3, R4, R5, R6
Changed lines of the file:
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@@
 <part name="GND1" library="supply1" library_urn="urn:adsk.eagle:library:371" deviceset="GND" device=""/>
 <part name="GND4" library="supply1" library_urn="urn:adsk.eagle:library:371" deviceset="GND" device=""/>
-<part name="C5" library="rcl" library_urn="urn:adsk.eagle:library:334" deviceset="C-EU" device="C0603" package3d_urn="urn:adsk.eagle:package:23616/2" value="1.5u"/>
-<part name="C6" library="rcl" library_urn="urn:adsk.eagle:library:334" deviceset="C-EU" device="C0603" package3d_urn="urn:adsk.eagle:package:23616/2" value="1.5u"/>
-<part name="R4" library="rcl" library_urn="urn:adsk.eagle:library:334" deviceset="R-EU_" device="R0603" package3d_urn="urn:adsk.eagle:package:23555/2" value="20"/>
+<part name="C3" library="rcl" library_urn="urn:adsk.eagle:library:334" deviceset="C-EU" device="C0603" package3d_urn="urn:adsk.eagle:package:23616/2" value="1.5u"/>
+<part name="C2" library="rcl" library_urn="urn:adsk.eagle:library:334" deviceset="C-EU" device="C0603" package3d_urn="urn:adsk.eagle:package:23616/2" value="1.5u"/>
+<part name="R5" library="rcl" library_urn="urn:adsk.eagle:library:334" deviceset="R-EU_" device="R0603" package3d_urn="urn:adsk.eagle:package:23555/2" value="20"/>
 <part name="GND6" library="supply1" library_urn="urn:adsk.eagle:library:371" deviceset="GND" device=""/>
 <part name="GND7" library="supply1" library_urn="urn:adsk.eagle:library:371" deviceset="GND" device=""/>
-<part name="C7" library="rcl" library_urn="urn:adsk.eagle:library:334" deviceset="C-EU" device="C0603" package3d_urn="urn:adsk.eagle:package:23616/2" value="10u"/>
+<part name="C1" library="rcl" library_urn="urn:adsk.eagle:library:334" deviceset="C-EU" device="C0603" package3d_urn="urn:adsk.eagle:package:23616/2" value="10u"/>
 <part name="GND8" library="supply1" library_urn="urn:adsk.eagle:library:371" deviceset="GND" device=""/>
 <part name="GND2" library="supply1" library_urn="urn:adsk.eagle:library:371" deviceset="GND" device=""/>
@@
 <part name="P+1" library="supply1" library_urn="urn:adsk.eagle:library:371" deviceset="+5V" device=""/>
 <part name="Q1" library="jonas_mosfet" library_urn="urn:adsk.eagle:library:2195717" deviceset="BSN20,215" device="" package3d_urn="urn:adsk.eagle:package:2195720/4"/>
-<part name="R3" library="rcl" library_urn="urn:adsk.eagle:library:334" deviceset="R-EU_" device="R0603" package3d_urn="urn:adsk.eagle:package:23555/2" value="4k7"/>
-<part name="R5" library="rcl" library_urn="urn:adsk.eagle:library:334" deviceset="R-EU_" device="R0603" package3d_urn="urn:adsk.eagle:package:23555/2" value="4k7"/>
+<part name="R6" library="rcl" library_urn="urn:adsk.eagle:library:334" deviceset="R-EU_" device="R0603" package3d_urn="urn:adsk.eagle:package:23555/2" value="4k7"/>
+<part name="R4" library="rcl" library_urn="urn:adsk.eagle:library:334" deviceset="R-EU_" device="R0603" package3d_urn="urn:adsk.eagle:package:23555/2" value="4k7"/>
 <part name="P+2" library="supply1" library_urn="urn:adsk.eagle:library:371" deviceset="+5V" device=""/>
 <part name="+3V5" library="supply1" library_urn="urn:adsk.eagle:library:371" deviceset="+3V3" device=""/>
@@
 <part name="JP2" library="SparkFun-Jumpers" library_urn="urn:adsk.eagle:library:528" deviceset="JUMPER-SMT_3_1-NC_TRACE" device="_SILK" package3d_urn="urn:adsk.eagle:package:39288/1" value=""/>
 <part name="LOGO1" library="SparkFun-Aesthetics" library_urn="urn:adsk.eagle:library:507" deviceset="OSHW-LOGO" device="M" package3d_urn="urn:adsk.eagle:package:37126/1"/>
-<part name="R6" library="rcl" library_urn="urn:adsk.eagle:library:334" deviceset="R-EU_" device="R0603" package3d_urn="urn:adsk.eagle:package:23555/2" value="10k"/>
+<part name="R3" library="rcl" library_urn="urn:adsk.eagle:library:334" deviceset="R-EU_" device="R0603" package3d_urn="urn:adsk.eagle:package:23555/2" value="10k"/>
 <part name="+3V6" library="supply1" library_urn="urn:adsk.eagle:library:371" deviceset="+3V3" device=""/>
 <part name="J3" library="SparkFun-Connectors" library_urn="urn:adsk.eagle:library:513" deviceset="CONN_03" device="SCREW-NS" package3d_urn="urn:adsk.eagle:package:38088/1"/>
@@
 <instance part="GND1" gate="1" x="12.7" y="104.14"/>
 <instance part="GND4" gate="1" x="48.26" y="88.9"/>
-<instance part="C5" gate="G$1" x="60.96" y="111.76"/>
-<instance part="C6" gate="G$1" x="53.34" y="111.76"/>
-<instance part="R4" gate="G$1" x="53.34" y="99.06" rot="R270"/>
+<instance part="C3" gate="G$1" x="60.96" y="111.76"/>
+<instance part="C2" gate="G$1" x="53.34" y="111.76"/>
+<instance part="R5" gate="G$1" x="53.34" y="99.06" rot="R270"/>
 <instance part="GND6" gate="1" x="60.96" y="88.9"/>
 <instance part="GND7" gate="1" x="53.34" y="88.9"/>
-<instance part="C7" gate="G$1" x="71.12" y="111.76"/>
+<instance part="C1" gate="G$1" x="71.12" y="111.76"/>
 <instance part="GND8" gate="1" x="71.12" y="88.9"/>
 <instance part="GND2" gate="1" x="152.4" y="38.1"/>
@@
 <instance part="P+1" gate="1" x="165.1" y="50.8"/>
 <instance part="Q1" gate="G$1" x="167.64" y="167.64" rot="R90"/>
-<instance part="R3" gate="G$1" x="177.8" y="177.8"/>
-<instance part="R5" gate="G$1" x="177.8" y="160.02"/>
+<instance part="R6" gate="G$1" x="177.8" y="177.8"/>
+<instance part="R4" gate="G$1" x="177.8" y="160.02"/>
 <instance part="P+2" gate="1" x="190.5" y="160.02" rot="R270"/>
 <instance part="+3V5" gate="G$1" x="190.5" y="177.8" rot="R270"/>
@@
 <instance part="JP2" gate="G$1" x="226.06" y="121.92" rot="R90"/>
 <instance part="LOGO1" gate="G$1" x="30.48" y="48.26"/>
-<instance part="R6" gate="G$1" x="81.28" y="45.72" rot="R90"/>
+<instance part="R3" gate="G$1" x="81.28" y="45.72" rot="R90"/>
 <instance part="+3V6" gate="G$1" x="81.28" y="55.88"/>
 <instance part="J3" gate="J$1" x="215.9" y="111.76"/>
@@
 <wire x1="71.12" y1="121.92" x2="71.12" y2="114.3" width="0.1524" layer="91"/>
 <junction x="48.26" y="121.92"/>
-<pinref part="C7" gate="G$1" pin="1"/>
+<pinref part="C1" gate="G$1" pin="1"/>
 </segment>
 <segment>
@@
 <wire x1="175.26" y1="170.18" x2="185.42" y2="170.18" width="0.1524" layer="91"/>
 <wire x1="185.42" y1="170.18" x2="185.42" y2="177.8" width="0.1524" layer="91"/>
-<pinref part="R3" gate="G$1" pin="2"/>
+<pinref part="R6" gate="G$1" pin="2"/>
 <wire x1="185.42" y1="177.8" x2="182.88" y2="177.8" width="0.1524" layer="91"/>
 <wire x1="185.42" y1="177.8" x2="187.96" y2="177.8" width="0.1524" layer="91"/>
@@
 </segment>
 <segment>
-<pinref part="R6" gate="G$1" pin="2"/>
+<pinref part="R3" gate="G$1" pin="2"/>
 <wire x1="81.28" y1="53.34" x2="81.28" y2="50.8" width="0.1524" layer="91"/>
 <pinref part="+3V6" gate="G$1" pin="+3V3"/>
@@
 </segment>
 <segment>
-<pinref part="R4" gate="G$1" pin="2"/>
+<pinref part="R5" gate="G$1" pin="2"/>
 <wire x1="53.34" y1="93.98" x2="53.34" y2="91.44" width="0.1524" layer="91"/>
 <pinref part="GND7" gate="1" pin="GND"/>
 </segment>
 <segment>
-<pinref part="C5" gate="G$1" pin="2"/>
+<pinref part="C3" gate="G$1" pin="2"/>
 <wire x1="60.96" y1="106.68" x2="60.96" y2="91.44" width="0.1524" layer="91"/>
 <pinref part="GND6" gate="1" pin="GND"/>
 </segment>
 <segment>
-<pinref part="C7" gate="G$1" pin="2"/>
+<pinref part="C1" gate="G$1" pin="2"/>
 <wire x1="71.12" y1="106.68" x2="71.12" y2="91.44" width="0.1524" layer="91"/>
 <pinref part="GND8" gate="1" pin="GND"/>
@@
 </segment>
 <segment>
-<pinref part="R6" gate="G$1" pin="1"/>
+<pinref part="R3" gate="G$1" pin="1"/>
 <wire x1="81.28" y1="40.64" x2="81.28" y2="38.1" width="0.1524" layer="91"/>
 <label x="81.28" y="38.1" size="1.016" layer="95" rot="R270" xref="yes"/>
@@
 <segment>
 <pinref part="U1" gate="G$1" pin="AVDD-PC"/>
-<pinref part="C6" gate="G$1" pin="1"/>
+<pinref part="C2" gate="G$1" pin="1"/>
 <wire x1="45.72" y1="116.84" x2="53.34" y2="116.84" width="0.1524" layer="91"/>
 <wire x1="53.34" y1="116.84" x2="53.34" y2="114.3" width="0.1524" layer="91"/>
@@
 <net name="N$6" class="0">
 <segment>
-<pinref part="C6" gate="G$1" pin="2"/>
-<pinref part="R4" gate="G$1" pin="1"/>
+<pinref part="C2" gate="G$1" pin="2"/>
+<pinref part="R5" gate="G$1" pin="1"/>
 <wire x1="53.34" y1="106.68" x2="53.34" y2="104.14" width="0.1524" layer="91"/>
 </segment>
@@
 <segment>
 <pinref part="U1" gate="G$1" pin="DVDD-PC"/>
-<pinref part="C5" gate="G$1" pin="1"/>
+<pinref part="C3" gate="G$1" pin="1"/>
 <wire x1="45.72" y1="119.38" x2="60.96" y2="119.38" width="0.1524" layer="91"/>
 <wire x1="60.96" y1="119.38" x2="60.96" y2="114.3" width="0.1524" layer="91"/>
@@
 </segment>
 <segment>
-<pinref part="R5" gate="G$1" pin="2"/>
+<pinref part="R4" gate="G$1" pin="2"/>
 <wire x1="182.88" y1="160.02" x2="187.96" y2="160.02" width="0.1524" layer="91"/>
 <pinref part="P+2" gate="1" pin="+5V"/>
@@
 <pinref part="Q1" gate="G$1" pin="S"/>
 <wire x1="170.18" y1="172.72" x2="170.18" y2="177.8" width="0.1524" layer="91"/>
-<pinref part="R3" gate="G$1" pin="1"/>
+<pinref part="R6" gate="G$1" pin="1"/>
 <wire x1="170.18" y1="177.8" x2="172.72" y2="177.8" width="0.1524" layer="91"/>
 <wire x1="170.18" y1="177.8" x2="170.18" y2="182.88" width="0.1524" layer="91"/>
@@
 <pinref part="Q1" gate="G$1" pin="D"/>
 <wire x1="170.18" y1="162.56" x2="170.18" y2="160.02" width="0.1524" layer="91"/>
-<pinref part="R5" gate="G$1" pin="1"/>
+<pinref part="R4" gate="G$1" pin="1"/>
 <wire x1="170.18" y1="160.02" x2="172.72" y2="160.02" width="0.1524" layer="91"/>
 <pinref part="JP1" gate="G$1" pin="2"/>

Commit message: 3d stuff
Parts:
- D1, D2, D3: device SparkFun-LED:WS2812B -> jonas_SparkFun-LED:WS2812B
- J1, J2: value (none) -> CONN_08; device SparkFun-Connectors:CONN_08LOCK_NO_SILK -> jonas_Sparkfun-Connectors:CONN_08
- J3: value (none) -> CONN_03SCREWTERMINAL-3.5MM-3-NS; device SparkFun-Connectors:CONN_03SCREW-NS -> jonas_Sparkfun-Connectors:CONN_03SCREWTERMINAL-3.5MM-3-NS
- JP1: value JUMPER-SMT_2_NC_TRACE_SILK -> JUMPER-SMT_2_NC_TRACE; device SparkFun-Jumpers:JUMPER-SMT_2_NC_TRACE_SILK -> jonas_SparkFun_Jumper:JUMPER-SMT_2_NC_TRACE
- JP2: value JUMPER-SMT_3_1-NC_TRACE_SILK -> JUMPER-SMT_3_1-NC_TRACE; device SparkFun-Jumpers:JUMPER-SMT_3_1-NC_TRACE_SILK -> jonas_SparkFun_Jumper:JUMPER-SMT_3_1-NC_TRACE
- LOGO1: value OSHW-LOGOM -> OSHW-LOGO; device SparkFun-Aesthetics:OSHW-LOGOM -> jonas_SparkFun-Aesthetics:OSHW-LOGO
Changed lines of the file:
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@@
 <?xml version="1.0" encoding="utf-8"?>
 <!DOCTYPE eagle SYSTEM "eagle.dtd">
-<eagle version="9.0.1">
+<eagle version="9.1.0">
 <drawing>
 <settings>
@@
 <part name="+3V3" library="supply1" library_urn="urn:adsk.eagle:library:371" deviceset="+3V3" device=""/>
 <part name="+3V4" library="supply1" library_urn="urn:adsk.eagle:library:371" deviceset="+3V3" device=""/>
-<part name="D1" library="SparkFun-LED" library_urn="urn:adsk.eagle:library:529" deviceset="WS2812B" device="" package3d_urn="urn:adsk.eagle:package:39369/1" value="WS2812B"/>
-<part name="D2" library="SparkFun-LED" library_urn="urn:adsk.eagle:library:529" deviceset="WS2812B" device="" package3d_urn="urn:adsk.eagle:package:39369/1" value="WS2812B"/>
-<part name="D3" library="SparkFun-LED" library_urn="urn:adsk.eagle:library:529" deviceset="WS2812B" device="" package3d_urn="urn:adsk.eagle:package:39369/1" value="WS2812B"/>
+<part name="D1" library="jonas_SparkFun-LED" library_urn="urn:adsk.eagle:library:3855694" deviceset="WS2812B" device="" package3d_urn="urn:adsk.eagle:package:3855696/2" value="WS2812B"/>
+<part name="D2" library="jonas_SparkFun-LED" library_urn="urn:adsk.eagle:library:3855694" deviceset="WS2812B" device="" package3d_urn="urn:adsk.eagle:package:3855696/2" value="WS2812B"/>
+<part name="D3" library="jonas_SparkFun-LED" library_urn="urn:adsk.eagle:library:3855694" deviceset="WS2812B" device="" package3d_urn="urn:adsk.eagle:package:3855696/2" value="WS2812B"/>
 <part name="P+1" library="supply1" library_urn="urn:adsk.eagle:library:371" deviceset="+5V" device=""/>
 <part name="Q1" library="jonas_mosfet" library_urn="urn:adsk.eagle:library:2195717" deviceset="BSN20,215" device="" package3d_urn="urn:adsk.eagle:package:2195720/4"/>
@@
 <part name="P+3" library="supply1" library_urn="urn:adsk.eagle:library:371" deviceset="+5V" device=""/>
 <part name="GND3" library="supply1" library_urn="urn:adsk.eagle:library:371" deviceset="GND" device=""/>
-<part name="J1" library="SparkFun-Connectors" library_urn="urn:adsk.eagle:library:513" deviceset="CONN_08" device="LOCK_NO_SILK" package3d_urn="urn:adsk.eagle:package:38147/1"/>
-<part name="J2" library="SparkFun-Connectors" library_urn="urn:adsk.eagle:library:513" deviceset="CONN_08" device="LOCK_NO_SILK" package3d_urn="urn:adsk.eagle:package:38147/1"/>
+<part name="J1" library="jonas_Sparkfun-Connectors" library_urn="urn:adsk.eagle:library:3855661" deviceset="CONN_08" device="" package3d_urn="urn:adsk.eagle:package:3855663/2" value=""/>
+<part name="J2" library="jonas_Sparkfun-Connectors" library_urn="urn:adsk.eagle:library:3855661" deviceset="CONN_08" device="" package3d_urn="urn:adsk.eagle:package:3855663/2" value=""/>
 <part name="P+4" library="supply1" library_urn="urn:adsk.eagle:library:371" deviceset="+5V" device=""/>
 <part name="GND5" library="supply1" library_urn="urn:adsk.eagle:library:371" deviceset="GND" device=""/>
-<part name="JP1" library="SparkFun-Jumpers" library_urn="urn:adsk.eagle:library:528" deviceset="JUMPER-SMT_2_NC_TRACE" device="_SILK" package3d_urn="urn:adsk.eagle:package:39281/1" value=""/>
-<part name="JP2" library="SparkFun-Jumpers" library_urn="urn:adsk.eagle:library:528" deviceset="JUMPER-SMT_3_1-NC_TRACE" device="_SILK" package3d_urn="urn:adsk.eagle:package:39288/1" value=""/>
-<part name="LOGO1" library="SparkFun-Aesthetics" library_urn="urn:adsk.eagle:library:507" deviceset="OSHW-LOGO" device="M" package3d_urn="urn:adsk.eagle:package:37126/1"/>
+<part name="JP1" library="jonas_SparkFun_Jumper" library_urn="urn:adsk.eagle:library:3855711" deviceset="JUMPER-SMT_2_NC_TRACE" device="" package3d_urn="urn:adsk.eagle:package:3855718/2" value="JUMPER-SMT_2_NC_TRACE"/>
+<part name="JP2" library="jonas_SparkFun_Jumper" library_urn="urn:adsk.eagle:library:3855711" deviceset="JUMPER-SMT_3_1-NC_TRACE" device="" package3d_urn="urn:adsk.eagle:package:3855713/2" value=""/>
+<part name="LOGO1" library="jonas_SparkFun-Aesthetics" library_urn="urn:adsk.eagle:library:3855705" deviceset="OSHW-LOGO" device="" package3d_urn="urn:adsk.eagle:package:3855707/2"/>
 <part name="R3" library="rcl" library_urn="urn:adsk.eagle:library:334" deviceset="R-EU_" device="R0603" package3d_urn="urn:adsk.eagle:package:23555/2" value="10k"/>
 <part name="+3V6" library="supply1" library_urn="urn:adsk.eagle:library:371" deviceset="+3V3" device=""/>
-<part name="J3" library="SparkFun-Connectors" library_urn="urn:adsk.eagle:library:513" deviceset="CONN_03" device="SCREW-NS" package3d_urn="urn:adsk.eagle:package:38088/1"/>
+<part name="J3" library="jonas_Sparkfun-Connectors" library_urn="urn:adsk.eagle:library:3855661" deviceset="CONN_03" device="SCREWTERMINAL-3.5MM-3-NS" package3d_urn="urn:adsk.eagle:package:3855668/2" value=""/>
 </parts>
 <sheets>
@@
 <instance part="R3" gate="G$1" x="81.28" y="45.72" rot="R90"/>
 <instance part="+3V6" gate="G$1" x="81.28" y="55.88"/>
-<instance part="J3" gate="J$1" x="215.9" y="111.76"/>
+<instance part="J3" gate="G$1" x="215.9" y="111.76"/>
 </instances>
 <busses>
@@
 <wire x1="226.06" y1="109.22" x2="226.06" y2="106.68" width="0.1524" layer="91"/>
 <pinref part="GND5" gate="1" pin="GND"/>
-<pinref part="J3" gate="J$1" pin="1"/>
+<pinref part="J3" gate="G$1" pin="1"/>
 </segment>
 </net>
@@
 <wire x1="233.68" y1="111.76" x2="233.68" y2="114.3" width="0.1524" layer="91"/>
 <pinref part="P+4" gate="1" pin="+5V"/>
-<pinref part="J3" gate="J$1" pin="2"/>
+<pinref part="J3" gate="G$1" pin="2"/>
 </segment>
 </net>
@@
 <wire x1="226.06" y1="114.3" x2="226.06" y2="116.84" width="0.1524" layer="91"/>
 <pinref part="JP2" gate="G$1" pin="2"/>
-<pinref part="J3" gate="J$1" pin="3"/>
-</segment>
-</net>
+<pinref part="J3" gate="G$1" pin="3"/>
+</segment>
+</net>
